Commit message: add depth camera

File: meshes/robot.urdf (robot description, URDF)
Before this commit: robot Walter, 13 links, 12 joints
Links:
- removed link lidar
- added link camera_ensamble, mass 0; collision mesh filename=package://meshes/camera.stl; visual mesh filename=package://meshes/camera.stl
- added link liddar, mass 1.3929559942642171233; collision mesh filename=package://meshes/lidar.stl; visual mesh filename=package://meshes/lidar.stl
- link cabeza_pecho: mass 32.542285355597933005 -> 32.542285355597947216
- link rueda: mass 1.2695552659388229522 -> 1.2695552659388233963
- link rueda_2: mass 1.2695552659388229522 -> 1.2695552659388233963
Joints:
- removed joint lidar_joint
- added joint camera: type fixed, parent cabeza_pecho, child camera_ensamble, origin xyz=0.16999999999999998446 -3.2959746043559334794e-17 -0.037499999999999977796 rpy=1.570796326794896558 -0 -1.570796326794896558, axis 0 0 1, limit effort=1.5 velocity=22
- added joint liddar_joint: type fixed, parent fijos_inferior, child liddar, origin xyz=-1.0408340855860842566e-17 -0.20637340124470737734 0.14700000000000001954 rpy=0 -0 -1.570796326794896558, axis 0 0 1, limit effort=1.5 velocity=22
