Commit message: add depth camera

File: urdf/walter.xacro (robot description, xacro)
@@ -12,5 +12,6 @@
             </geometry>
             <material name="torso_material">
-                <color rgba="0.91764705882352937127 0.91764705882352937127 0.91764705882352937127 1.0" />
+                <color
+                    rgba="0.91764705882352937127 0.91764705882352937127 0.91764705882352937127 1.0" />
             </material>
         </visual>
@@ -22,7 +23,10 @@
         </collision>
         <inertial>
-            <origin xyz="3.5366736310120974436e-06 1.016494425031958053e-06 -0.10404383296951648374" rpy="0 0 0" />
+            <origin xyz="3.5366736310120974436e-06 1.016494425031958053e-06 -0.10404383296951648374"
+                rpy="0 0 0" />
             <mass value="37.981250382069397631" />
-            <inertia ixx="0.93147768307078449013" ixy="-1.0314156922500628319e-05" ixz="-3.7114421258874762019e-06" iyy="0.93168041764494147206" iyz="-1.7562940793422002905e-06" izz="0.68744587515199118144" />
+            <inertia ixx="0.93147768307078449013" ixy="-1.0314156922500628319e-05"
+                ixz="-3.7114421258874762019e-06" iyy="0.93168041764494147206"
+                iyz="-1.7562940793422002905e-06" izz="0.68744587515199118144" />
         </inertial>
     </link>
@@ -34,5 +38,6 @@
             </geometry>
             <material name="pecho_material">
-                <color rgba="0.90196078431372550543 0.90196078431372550543 0.90196078431372550543 1.0" />
+                <color
+                    rgba="0.90196078431372550543 0.90196078431372550543 0.90196078431372550543 1.0" />
             </material>
         </visual>
@@ -44,14 +49,17 @@
         </collision>
         <visual>
-            <origin xyz="0.035000000000000003331 -2.6020852139652106416e-18 -0.26999999999999979572" rpy="3.141592653589793116 -7.7355025826137686325e-17 -7.3589012180439136812e-17" />
+            <origin xyz="0.035000000000000003331 -2.6020852139652106416e-18 -0.26999999999999979572"
+                rpy="3.141592653589793116 -7.7355025826137686325e-17 -7.3589012180439136812e-17" />
             <geometry>
                 <mesh filename="package://walter_description/meshes/cabeza.stl" />
             </geometry>
             <material name="cabeza_material">
-                <color rgba="0.90196078431372550543 0.90196078431372550543 0.90196078431372550543 1.0" />
-            </material>
-        </visual>
-        <collision>
-            <origin xyz="0.035000000000000003331 -2.6020852139652106416e-18 -0.26999999999999979572" rpy="3.141592653589793116 -7.7355025826137686325e-17 -7.3589012180439136812e-17" />
+                <color
+                    rgba="0.90196078431372550543 0.90196078431372550543 0.90196078431372550543 1.0" />
+            </material>
+        </visual>
+        <collision>
+            <origin xyz="0.035000000000000003331 -2.6020852139652106416e-18 -0.26999999999999979572"
+                rpy="3.141592653589793116 -7.7355025826137686325e-17 -7.3589012180439136812e-17" />
             <geometry>
                 <mesh filename="package://walter_description/meshes/cabeza.stl" />
@@ -59,14 +67,17 @@
         </collision>
         <visual>
-            <origin xyz="5.1223973916507838371e-18 0.19500000000000003442 -0.017780000000000018012" rpy="3.141592653589793116 -6.0722997586192119681e-17 -3.141592653589793116" />
+            <origin xyz="5.1223973916507838371e-18 0.19500000000000003442 -0.017780000000000018012"
+                rpy="3.141592653589793116 -6.0722997586192119681e-17 -3.141592653589793116" />
             <geometry>
                 <mesh filename="package://walter_description/meshes/brazo1.stl" />
             </geometry>
             <material name="brazo1_material">
-                <color rgba="0.90196078431372550543 0.90196078431372550543 0.90196078431372550543 1.0" />
-            </material>
-        </visual>
-        <collision>
-            <origin xyz="5.1223973916507838371e-18 0.19500000000000003442 -0.017780000000000018012" rpy="3.141592653589793116 -6.0722997586192119681e-17 -3.141592653589793116" />
+                <color
+                    rgba="0.90196078431372550543 0.90196078431372550543 0.90196078431372550543 1.0" />
+            </material>
+        </visual>
+        <collision>
+            <origin xyz="5.1223973916507838371e-18 0.19500000000000003442 -0.017780000000000018012"
+                rpy="3.141592653589793116 -6.0722997586192119681e-17 -3.141592653589793116" />
             <geometry>
                 <mesh filename="package://walter_description/meshes/brazo1.stl" />
@@ -74,14 +85,19 @@
         </collision>
         <visual>
-            <origin xyz="-7.6387795496199423289e-18 -0.18000000000000002109 -0.017780000000000018012" rpy="3.141592653589793116 -0 -3.141592653589793116" />
+            <origin
+                xyz="-7.6387795496199423289e-18 -0.18000000000000002109 -0.017780000000000018012"
+                rpy="3.141592653589793116 -0 -3.141592653589793116" />
             <geometry>
                 <mesh filename="package://walter_description/meshes/brazo1.stl" />
             </geometry>
             <material name="brazo1_material">
-                <color rgba="0.90196078431372550543 0.90196078431372550543 0.90196078431372550543 1.0" />
-            </material>
-        </visual>
-        <collision>
-            <origin xyz="-7.6387795496199423289e-18 -0.18000000000000002109 -0.017780000000000018012" rpy="3.141592653589793116 -0 -3.141592653589793116" />
+                <color
+                    rgba="0.90196078431372550543 0.90196078431372550543 0.90196078431372550543 1.0" />
+            </material>
+        </visual>
+        <collision>
+            <origin
+                xyz="-7.6387795496199423289e-18 -0.18000000000000002109 -0.017780000000000018012"
+                rpy="3.141592653589793116 -0 -3.141592653589793116" />
             <geometry>
                 <mesh filename="package://walter_description/meshes/brazo1.stl" />
@@ -89,12 +105,18 @@
         </collision>
         <inertial>
-            <origin xyz="0.0027210420105864435193 -0.00020045946930026377016 -0.096581144323558784648" rpy="0 0 0" />
+            <origin
+                xyz="0.0027210420105864435193 -0.00020045946930026377016 -0.096581144323558784648"
+                rpy="0 0 0" />
             <mass value="32.542285355597933005" />
-            <inertia ixx="0.45532393141777993684" ixy="-3.1430516357851701753e-05" ixz="0.0062540021383989292947" iyy="0.40737380981547899328" iyz="-0.0011563569028698351959" izz="0.3885002478865637876" />
+            <inertia ixx="0.45532393141777993684" ixy="-3.1430516357851701753e-05"
+                ixz="0.0062540021383989292947" iyy="0.40737380981547899328"
+                iyz="-0.0011563569028698351959" izz="0.3885002478865637876" />
         </inertial>
     </link>
     <link name="pantalla">
         <visual>
-            <origin xyz="-4.1633363423443370266e-17 -0.0063773533988664699024 -0.0010000000000000008882" rpy="-1.570796326794896558 -1.570796326794896558 0" />
+            <origin
+                xyz="-4.1633363423443370266e-17 -0.0063773533988664699024 -0.0010000000000000008882"
+                rpy="-1.570796326794896558 -1.570796326794896558 0" />
             <geometry>
                 <mesh filename="package://walter_description/meshes/pantalla.stl" />
@@ -105,5 +127,7 @@
         </visual>
         <collision>
-            <origin xyz="-4.1633363423443370266e-17 -0.0063773533988664699024 -0.0010000000000000008882" rpy="-1.570796326794896558 -1.570796326794896558 0" />
+            <origin
+                xyz="-4.1633363423443370266e-17 -0.0063773533988664699024 -0.0010000000000000008882"
+                rpy="-1.570796326794896558 -1.570796326794896558 0" />
             <geometry>
                 <mesh filename="package://walter_description/meshes/pantalla.stl" />
@@ -111,12 +135,16 @@
         </collision>
         <inertial>
-            <origin xyz="-5.9224247552555778029e-18 -9.7144514654701184961e-17 -0.00050000000000000087777" rpy="0 0 0" />
+            <origin
+                xyz="-5.9224247552555778029e-18 -9.7144514654701184961e-17 -0.00050000000000000087777"
+                rpy="0 0 0" />
             <mass value="0.052708425382244711299" />
-            <inertia ixx="8.7518885294316788753e-05" ixy="0" ixz="7.3163984344922236004e-37" iyy="0.00012648147131393697238" iyz="0" izz="0.00021399157187069003548" />
+            <inertia ixx="8.7518885294316788753e-05" ixy="0" ixz="7.3163984344922236004e-37"
+                iyy="0.00012648147131393697238" iyz="0" izz="0.00021399157187069003548" />
         </inertial>
     </link>
     <link name="ojo_der">
         <visual>
-            <origin xyz="0.049288699999999997792 -0.015239999999999920277 -0.0030000000000000026645" rpy="-1.570796326794896558 4.5998421556777242306e-33 0" />
+            <origin xyz="0.049288699999999997792 -0.015239999999999920277 -0.0030000000000000026645"
+                rpy="-1.570796326794896558 4.5998421556777242306e-33 0" />
             <geometry>
                 <mesh filename="package://walter_description/meshes/ojo1.stl" />
@@ -127,5 +155,6 @@
         </visual>
         <collision>
-            <origin xyz="0.049288699999999997792 -0.015239999999999920277 -0.0030000000000000026645" rpy="-1.570796326794896558 4.5998421556777242306e-33 0" />
+            <origin xyz="0.049288699999999997792 -0.015239999999999920277 -0.0030000000000000026645"
+                rpy="-1.570796326794896558 4.5998421556777242306e-33 0" />
             <geometry>
                 <mesh filename="package://walter_description/meshes/ojo1.stl" />
@@ -133,12 +162,17 @@
         </collision>
         <inertial>
-            <origin xyz="-2.1725723654830719767e-07 -4.1358975869099090517e-07 -0.0015000000000000024165" rpy="0 0 0" />
+            <origin
+                xyz="-2.1725723654830719767e-07 -4.1358975869099090517e-07 -0.0015000000000000024165"
+                rpy="0 0 0" />
             <mass value="0.016158389381498900611" />
-            <inertia ixx="6.2099029968954678815e-06" ixy="-1.3050423685354312141e-10" ixz="-1.2937429533846938739e-14" iyy="1.6722806386780241734e-06" iyz="7.6244819049309471189e-38" izz="7.8579465371037161289e-06" />
+            <inertia ixx="6.2099029968954678815e-06" ixy="-1.3050423685354312141e-10"
+                ixz="-1.2937429533846938739e-14" iyy="1.6722806386780241734e-06"
+                iyz="7.6244819049309471189e-38" izz="7.8579465371037161289e-06" />
         </inertial>
     </link>
     <link name="ojo_izq">
         <visual>
-            <origin xyz="-0.04928870000000001167 -0.015239999999999920277 -0.0030000000000000026645" rpy="-1.570796326794896558 4.5998421556777242306e-33 0" />
+            <origin xyz="-0.04928870000000001167 -0.015239999999999920277 -0.0030000000000000026645"
+                rpy="-1.570796326794896558 4.5998421556777242306e-33 0" />
             <geometry>
                 <mesh filename="package://walter_description/meshes/ojo2.stl" />
@@ -149,5 +183,6 @@
         </visual>
         <collision>
-            <origin xyz="-0.04928870000000001167 -0.015239999999999920277 -0.0030000000000000026645" rpy="-1.570796326794896558 4.5998421556777242306e-33 0" />
+            <origin xyz="-0.04928870000000001167 -0.015239999999999920277 -0.0030000000000000026645"
+                rpy="-1.570796326794896558 4.5998421556777242306e-33 0" />
             <geometry>
                 <mesh filename="package://walter_description/meshes/ojo2.stl" />
@@ -155,21 +190,28 @@
         </collision>
         <inertial>
-            <origin xyz="-2.1725723654136830376e-07 -4.1358975869446035212e-07 -0.0015000000000000026333" rpy="0 0 0" />
+            <origin
+                xyz="-2.1725723654136830376e-07 -4.1358975869446035212e-07 -0.0015000000000000026333"
+                rpy="0 0 0" />
             <mass value="0.016158389381498900611" />
-            <inertia ixx="6.2099029968954644934e-06" ixy="-1.3050423685349602382e-10" ixz="-1.2937429532790463083e-14" iyy="1.6722806386780231146e-06" iyz="7.6244819049309418987e-38" izz="7.8579465371037110467e-06" />
+            <inertia ixx="6.2099029968954644934e-06" ixy="-1.3050423685349602382e-10"
+                ixz="-1.2937429532790463083e-14" iyy="1.6722806386780231146e-06"
+                iyz="7.6244819049309418987e-38" izz="7.8579465371037110467e-06" />
         </inertial>
     </link>
     <link name="fijos_inferior">
         <visual>
-            <origin xyz="-3.6429192995512948983e-17 0.20637340124470746061 0.010000000000000000208" rpy="0 -0 0" />
+            <origin xyz="-3.6429192995512948983e-17 0.20637340124470746061 0.010000000000000000208"
+                rpy="0 -0 0" />
             <geometry>
                 <mesh filename="package://walter_description/meshes/eje_caster.stl" />
             </geometry>
             <material name="eje_caster_material">
-                <color rgba="0.49803921568627451677 0.49803921568627451677 0.49803921568627451677 1.0" />
-            </material>
-        </visual>
-        <collision>
-            <origin xyz="-3.6429192995512948983e-17 0.20637340124470746061 0.010000000000000000208" rpy="0 -0 0" />
+                <color
+                    rgba="0.49803921568627451677 0.49803921568627451677 0.49803921568627451677 1.0" />
+            </material>
+        </visual>
+        <collision>
+            <origin xyz="-3.6429192995512948983e-17 0.20637340124470746061 0.010000000000000000208"
+                rpy="0 -0 0" />
             <geometry>
                 <mesh filename="package://walter_description/meshes/eje_caster.stl" />
@@ -177,5 +219,6 @@
         </collision>
         <visual>
-            <origin xyz="0 -0.13017340124470738738 0.12430000000000002158" rpy="3.141592653589793116 -0 0" />
+            <origin xyz="0 -0.13017340124470738738 0.12430000000000002158"
+                rpy="3.141592653589793116 -0 0" />
             <geometry>
                 <mesh filename="package://walter_description/meshes/bloque_1.stl" />
@@ -186,5 +229,6 @@
         </visual>
         <collision>
-            <origin xyz="0 -0.13017340124470738738 0.12430000000000002158" rpy="3.141592653589793116 -0 0" />
+            <origin xyz="0 -0.13017340124470738738 0.12430000000000002158"
+                rpy="3.141592653589793116 -0 0" />
             <geometry>
                 <mesh filename="package://walter_description/meshes/bloque_1.stl" />
@@ -192,5 +236,6 @@
         </collision>
         <visual>
-            <origin xyz="0 0.13017340124470744289 0.12430000000000002158" rpy="3.141592653589793116 -0 0" />
+            <origin xyz="0 0.13017340124470744289 0.12430000000000002158"
+                rpy="3.141592653589793116 -0 0" />
             <geometry>
                 <mesh filename="package://walter_description/meshes/bloque_1.stl" />
@@ -201,5 +246,6 @@
         </visual>
         <collision>
-            <origin xyz="0 0.13017340124470744289 0.12430000000000002158" rpy="3.141592653589793116 -0 0" />
+            <origin xyz="0 0.13017340124470744289 0.12430000000000002158"
+                rpy="3.141592653589793116 -0 0" />
             <geometry>
                 <mesh filename="package://walter_description/meshes/bloque_1.stl" />
@@ -227,5 +273,6 @@
             </geometry>
             <material name="protector_1_material">
-                <color rgba="0.91764705882352937127 0.91764705882352937127 0.91764705882352937127 1.0" />
+                <color
+                    rgba="0.91764705882352937127 0.91764705882352937127 0.91764705882352937127 1.0" />
             </material>
         </visual>
@@ -252,14 +299,17 @@
         </collision>
         <visual>
-            <origin xyz="0.21499999999999996891 1.1102230246251565404e-16 0.14700000000000001954" rpy="0 -0 0" />
+            <origin xyz="0.21499999999999996891 1.1102230246251565404e-16 0.14700000000000001954"
+                rpy="0 -0 0" />
             <geometry>
                 <mesh filename="package://walter_description/meshes/varilla.stl" />
             </geometry>
             <material name="varilla_material">
-                <color rgba="0.90196078431372550543 0.90196078431372550543 0.90196078431372550543 1.0" />
-            </material>
-        </visual>
-        <collision>
-            <origin xyz="0.21499999999999996891 1.1102230246251565404e-16 0.14700000000000001954" rpy="0 -0 0" />
+                <color
+                    rgba="0.90196078431372550543 0.90196078431372550543 0.90196078431372550543 1.0" />
+            </material>
+        </visual>
+        <collision>
+            <origin xyz="0.21499999999999996891 1.1102230246251565404e-16 0.14700000000000001954"
+                rpy="0 -0 0" />
             <geometry>
                 <mesh filename="package://walter_description/meshes/varilla.stl" />
@@ -267,14 +317,17 @@
         </collision>
         <visual>
-            <origin xyz="-3.7024656657773666662e-17 -0.2063734012447074051 0.010000000000000000208" rpy="0 -0 1.570796326794896558" />
+            <origin xyz="-3.7024656657773666662e-17 -0.2063734012447074051 0.010000000000000000208"
+                rpy="0 -0 1.570796326794896558" />
             <geometry>
                 <mesh filename="package://walter_description/meshes/eje_caster.stl" />
             </geometry>
             <material name="eje_caster_material">
-                <color rgba="0.49803921568627451677 0.49803921568627451677 0.49803921568627451677 1.0" />
-            </material>
-        </visual>
-        <collision>
-            <origin xyz="-3.7024656657773666662e-17 -0.2063734012447074051 0.010000000000000000208" rpy="0 -0 1.570796326794896558" />
+                <color
+                    rgba="0.49803921568627451677 0.49803921568627451677 0.49803921568627451677 1.0" />
+            </material>
+        </visual>
+        <collision>
+            <origin xyz="-3.7024656657773666662e-17 -0.2063734012447074051 0.010000000000000000208"
+                rpy="0 -0 1.570796326794896558" />
             <geometry>
                 <mesh filename="package://walter_description/meshes/eje_caster.stl" />
@@ -297,14 +350,19 @@
         </collision>
         <visual>
-            <origin xyz="-5.8090702579312169077e-17 -0.17462340124470740466 -0.036458000000000004293" rpy="0 -0 -1.570796326794896558" />
+            <origin
+                xyz="-5.8090702579312169077e-17 -0.17462340124470740466 -0.036458000000000004293"
+                rpy="0 -0 -1.570796326794896558" />
             <geometry>
                 <mesh filename="package://walter_description/meshes/base_caster.stl" />
             </geometry>
             <material name="base_caster_material">
-                <color rgba="0.49803921568627451677 0.49803921568627451677 0.49803921568627451677 1.0" />
-            </material>
-        </visual>
-        <collision>
-            <origin xyz="-5.8090702579312169077e-17 -0.17462340124470740466 -0.036458000000000004293" rpy="0 -0 -1.570796326794896558" />
+                <color
+                    rgba="0.49803921568627451677 0.49803921568627451677 0.49803921568627451677 1.0" />
+            </material>
+        </visual>
+        <collision>
+            <origin
+                xyz="-5.8090702579312169077e-17 -0.17462340124470740466 -0.036458000000000004293"
+                rpy="0 -0 -1.570796326794896558" />
             <geometry>
                 <mesh filename="package://walter_description/meshes/base_caster.stl" />
@@ -312,14 +370,17 @@
         </collision>
         <visual>
-            <origin xyz="-3.6429192995512948983e-17 0.20637340124470746061 -0.036458000000000004293" rpy="0 -0 -1.570796326794896558" />
+            <origin xyz="-3.6429192995512948983e-17 0.20637340124470746061 -0.036458000000000004293"
+                rpy="0 -0 -1.570796326794896558" />
             <geometry>
                 <mesh filename="package://walter_description/meshes/base_caster.stl" />
             </geometry>
             <material name="base_caster_material">
-                <color rgba="0.49803921568627451677 0.49803921568627451677 0.49803921568627451677 1.0" />
-            </material>
-        </visual>
-        <collision>
-            <origin xyz="-3.6429192995512948983e-17 0.20637340124470746061 -0.036458000000000004293" rpy="0 -0 -1.570796326794896558" />
+                <color
+                    rgba="0.49803921568627451677 0.49803921568627451677 0.49803921568627451677 1.0" />
+            </material>
+        </visual>
+        <collision>
+            <origin xyz="-3.6429192995512948983e-17 0.20637340124470746061 -0.036458000000000004293"
+                rpy="0 -0 -1.570796326794896558" />
             <geometry>
                 <mesh filename="package://walter_description/meshes/base_caster.stl" />
@@ -332,5 +393,6 @@
             </geometry>
             <material name="protector_2_material">
-                <color rgba="0.91764705882352937127 0.91764705882352937127 0.91764705882352937127 1.0" />
+                <color
+                    rgba="0.91764705882352937127 0.91764705882352937127 0.91764705882352937127 1.0" />
             </material>
         </visual>
@@ -362,5 +424,6 @@
             </geometry>
             <material name="varilla_material">
-                <color rgba="0.90196078431372550543 0.90196078431372550543 0.90196078431372550543 1.0" />
+                <color
+                    rgba="0.90196078431372550543 0.90196078431372550543 0.90196078431372550543 1.0" />
             </material>
         </visual>
@@ -372,7 +435,10 @@
         </collision>
         <inertial>
-            <origin xyz="-0.0001122829556244791323 0.00095701728817520386253 0.06340814145131191959" rpy="0 0 0" />
+            <origin xyz="-0.0001122829556244791323 0.00095701728817520386253 0.06340814145131191959"
+                rpy="0 0 0" />
             <mass value="23.36660405251430106" />
-            <inertia ixx="0.51144499730725068165" ixy="0.00049729430174384086413" ixz="-0.00026868006102055019433" iyy="0.19831524554747295697" iyz="0.0015452552216950622005" izz="0.64852411735235737655" />
+            <inertia ixx="0.51144499730725068165" ixy="0.00049729430174384086413"
+                ixz="-0.00026868006102055019433" iyy="0.19831524554747295697"
+                iyz="0.0015452552216950622005" izz="0.64852411735235737655" />
         </inertial>
     </link>
@@ -394,7 +460,10 @@
         </collision>
         <inertial>
-            <origin xyz="-5.1779413895018431277e-67 1.6788122156820142359e-18 -0.012700000000000001218" rpy="0 0 0" />
+            <origin
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