Commit message: add depth camera

File: urdf/walter_gazebo.xacro (robot description, xacro)
@@ -11,8 +11,14 @@
     <preserveFixedJoint>true</preserveFixedJoint>
   </gazebo>
-  <gazebo reference="lidar">
-    <selfCollide>true</selfCollide>
-    <gravity>true</gravity>
-    <material>Gazebo/Red</material>
+  <gazebo reference="liddar">
+    <selfCollide>true</selfCollide>
+    <gravity>true</gravity>
+    <material>Gazebo/Blue</material>
+    <preserveFixedJoint>true</preserveFixedJoint>
+  </gazebo>
+  <gazebo reference="camera_ensamble">
+    <selfCollide>true</selfCollide>
+    <gravity>true</gravity>
+    <material>Gazebo/Blue</material>
     <preserveFixedJoint>true</preserveFixedJoint>
   </gazebo>
@@ -164,4 +170,29 @@
     </sensor>
   </gazebo>
+  <!-- camera plugging-->
+  <gazebo reference="camera_ensamble">
+    <sensor name="intel_realsense_r200_depth" type="depth">
+      <always_on>1</always_on>
+      <update_rate>1</update_rate>
+      <pose>0 0 0 0 0 0</pose>
+      <camera name="realsense_depth_camera">
+      </camera>
+      <plugin name="intel_realsense_r200_depth_driver" filename="libgazebo_ros_camera.so">
+        <ros>
+          <!--
+              <argument>custom_camera/image_raw:=custom_camera/custom_image</argument>
+              <argument>custom_camera/image_depth:=custom_camera/custom_image_depth</argument>
+              <argument>custom_camera/camera_info:=custom_camera/custom_info_raw</argument>
+              <argument>custom_camera/camera_info_depth:=custom_camera/custom_info_depth</argument>
+              <argument>custom_camera/points:=custom_camera/custom_points</argument>
+        -->
+        </ros>
+        <camera_name>intel_realsense_r200_depth</camera_name>
+        <frame_name>camera_link_optical</frame_name>
+        <hack_baseline>0.07</hack_baseline>
+        <min_depth>0.001</min_depth>
+      </plugin>
+    </sensor>
+  </gazebo>
   <!-- Diferencial drive controladores-->
   <gazebo>
