Commit message: fix axis camera

File: urdf/walter.xacro (robot description, xacro)
@@ -713,6 +713,8 @@
     </joint>
     <joint name="camera" type="fixed">
-        <origin xyz="0.16999999999999998446 -3.2959746043559334794e-17 -0.037499999999999977796"
-            rpy="1.570796326794896558 -0 -1.570796326794896558" />
+        <!-- <origin xyz="0.16999999999999998446 -3.2959746043559334794e-17 -0.037499999999999977796"
+            rpy="1.570796326794896558 -0 -1.570796326794896558" /> -->
+            <origin xyz="0.13 -3.2959746043559334794e-17 -0.037499999999999977796"
+            rpy="${pi} 0 0" />
         <parent link="cabeza_pecho" />
         <child link="camera_ensamble" />
@@ -724,6 +726,6 @@
         <parent link="camera_ensamble" />
         <child link="camera_link_optical" />
+        <!-- <origin xyz="0 0 0" rpy="${-pi/2} 0 ${-pi/2}" /> -->
         <origin xyz="0 0 0" rpy="${-pi/2} 0 ${-pi/2}" />
-        <!-- <origin xyz="0 0 0" rpy="0 0 0" /> -->
     </joint>
     <joint name="rueda_izquierda" type="continuous">

File: urdf/walter_gazebo.xacro (robot description, xacro)
@@ -175,9 +175,16 @@
       <always_on>1</always_on>
       <update_rate>1</update_rate>
-      <pose>0 0 0 0 0 0</pose>
+      <pose>0 0 0 3.14159 0 -1.57</pose>
       <camera name="realsense_depth_camera">
       </camera>
       <plugin name="intel_realsense_r200_depth_driver" filename="libgazebo_ros_camera.so">
         <ros>
+          <image>
+            <format>B8G8R8</format>
+          </image>
+          <clip>
+            <near>0.05</near>
+            <far>8.0</far>
+          </clip>
           <!--
               <argument>custom_camera/image_raw:=custom_camera/custom_image</argument>

Commit message: add right odom frame and depth camera

File: urdf/walter.xacro (robot description, xacro)
@@ -1,4 +1,4 @@
 <?xml version="1.0"?>
-<robot name="Walter"
+<robot name="walter"
     xmlns:xacro="http://www.ros.org/wiki/xacro">
     <xacro:include filename="$(find walter_description)/urdf/walter_gazebo.xacro" />
@@ -713,7 +713,8 @@
     </joint>
     <joint name="camera" type="fixed">
-        <!-- <origin xyz="0.16999999999999998446 -3.2959746043559334794e-17 -0.037499999999999977796"
+        <!-- <origin xyz="0.16999999999999998446 -3.2959746043559334794e-17
+        -0.037499999999999977796"
             rpy="1.570796326794896558 -0 -1.570796326794896558" /> -->
-            <origin xyz="0.13 -3.2959746043559334794e-17 -0.037499999999999977796"
+        <origin xyz="0.13 -3.2959746043559334794e-17 -0.037499999999999977796"
             rpy="${pi} 0 0" />
         <parent link="cabeza_pecho" />
@@ -819,3 +820,21 @@
         <joint_properties friction="0.0" />
     </joint>
+   <transmission name="transmission_rueda_izquierda">
+        <type>transmission_interface/SimpleTransmission</type>
+        <joint name="rueda_izquierda">
+            <hardwareInterface>hardware_interface/VelocityJointInterface</hardwareInterface>
+        </joint>
+        <actuator name="motor_rueda_izquierda">
+            <hardwareInterface>hardware_interface/ActuatorInterface</hardwareInterface>
+        </actuator>
+    </transmission>
+    <transmission name="transmission_rueda_derecha">
+        <type>transmission_interface/SimpleTransmission</type>
+        <joint name="rueda_derecha">
+            <hardwareInterface>hardware_interface/VelocityJointInterface</hardwareInterface>
+        </joint>
+        <actuator name="motor_rueda_derecha">
+            <hardwareInterface>hardware_interface/ActuatorInterface</hardwareInterface>
+        </actuator>
+    </transmission>
 </robot>

File: urdf/walter_gazebo.xacro (robot description, xacro)
@@ -1,4 +1,4 @@
 <?xml version="1.0"?>
-<robot name="Walter"
+<robot name="walter"
   xmlns:xacro="http://www.ros.org/wiki/xacro">
   <!-- Gazebo plugings -->
@@ -104,5 +104,5 @@
   </gazebo>
   <gazebo reference="rueda">
-    <mu1 value="100000.0" />
+    <mu1 value="1000.0" />
     <mu2 value="100000.0" />
     <kp value="10000000.0" />
@@ -111,5 +111,5 @@
   </gazebo>
   <gazebo reference="rueda_2">
-    <mu1 value="100000.0" />
+    <mu1 value="1000.0" />
     <mu2 value="100000.0" />
     <kp value="10000000.0" />
@@ -174,5 +174,5 @@
     <sensor name="intel_realsense_r200_depth" type="depth">
       <always_on>1</always_on>
-      <update_rate>1</update_rate>
+      <update_rate>30</update_rate>
       <pose>0 0 0 3.14159 0 -1.57</pose>
       <camera name="realsense_depth_camera">
@@ -185,5 +185,5 @@
           <clip>
             <near>0.05</near>
-            <far>8.0</far>
+            <far>5.0</far>
           </clip>
           <!--
@@ -198,5 +198,6 @@
         <frame_name>camera_link_optical</frame_name>
         <hack_baseline>0.07</hack_baseline>
-        <min_depth>0.001</min_depth>
+        <min_depth>0.01</min_depth>
+        <max_depth>50.0</max_depth>
       </plugin>
     </sensor>
@@ -205,4 +206,6 @@
   <gazebo>
     <plugin name="gazebo_ros2_control" filename="libgazebo_ros2_control.so">
+      <robot_param>robot_description</robot_param>
+      <robot_param_node>robot_state_publisher</robot_param_node>
       <parameters>$(find walter_description)/config/controllers.yaml</parameters>
       <ros>
@@ -211,4 +214,5 @@
       </ros>
     </plugin>
+    <plugin name="gazebo_ros_state" filename="libgazebo_ros_state.so" />
   </gazebo>
 </robot>
